File: schémas/schémas.kicad_sch (KiCad schematic)
At the start: 16 parts, among them J1 Conn_01x04, J2 Conn_01x04, J3 Conn_01x08, J4 Conn_01x08, J5 Conn_01x03, SW1 SW_Push_Dual, SW2 SW_Push_Dual, U1 ESP32-C3_SUPERMINI_SMD, U2 DHT22, U3 LTC-4627JS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

Commit message: feat: added button to diagram
Parts:
- removed SW1: SW_Push_Dual, Button_Switch_THT:SW_SPST_Omron_B3F-50xx, symbol Switch:SW_Push_Dual
- added SW3: SW_Push, Button_Switch_THT:SW_Tactile_SKHH_Angled, symbol Switch:SW_Push
Connections:
- net GND: now also SW3.2
- net at J4.8 (Pin_8), U5.21 (GPIO21): now also SW3.1
- no-connect marks 18 -> 16
Changed lines of the file:
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@@
 	(paper "A4")
-	(junction
-		(at 118.11 76.2)
-		(diameter 0)
-		(color 0 0 0 0)
-	)
 	(junction
 		(at 160.02 81.28)
@@
 	)
 	(junction
+		(at 118.11 93.98)
+		(diameter 0)
+		(color 0 0 0 0)
+	)
+	(junction
 		(at 91.44 88.9)
 		(diameter 0)
@@
 	)
 	(no_connect
-		(at 120.65 59.69)
-	)
-	(no_connect
 		(at -156.21 17.78)
 	)
@@
 	)
 	(no_connect
-		(at 115.57 69.85)
-	)
-	(no_connect
 		(at -120.65 5.08)
 	)
@@
 	(wire
 		(pts
-			(xy 115.57 59.69) (xy 115.57 55.88)
-		)
-		(stroke
-			(width 0)
-			(type default)
-		)
-	)
-	(wire
-		(pts
 			(xy 200.66 96.52) (xy 195.58 96.52)
 		)
@@
 	(wire
 		(pts
-			(xy 115.57 55.88) (xy 107.95 55.88)
+			(xy 69.85 99.06) (xy 76.2 99.06)
 		)
 		(stroke
@@
 	(wire
 		(pts
-			(xy 120.65 71.12) (xy 120.65 69.85)
-		)
-		(stroke
-			(width 0)
-			(type default)
-		)
-	)
-	(wire
-		(pts
 			(xy 198.12 85.09) (xy 200.66 85.09)
 		)
@@
 	(wire
 		(pts
+			(xy 200.66 90.17) (xy 200.66 96.52)
+		)
+		(stroke
+			(width 0)
+			(type default)
+		)
+	)
+	(wire
+		(pts
+			(xy 116.84 39.37) (xy 124.46 39.37)
+		)
+		(stroke
+			(width 0)
+			(type default)
+		)
+	)
+	(wire
+		(pts
+			(xy 71.12 52.07) (xy 71.12 54.61)
+		)
+		(stroke
+			(width 0)
+			(type default)
+		)
+	)
+	(wire
+		(pts
 			(xy 118.11 76.2) (xy 121.92 76.2)
 		)
@@
 	(wire
 		(pts
-			(xy 113.03 76.2) (xy 118.11 76.2)
-		)
-		(stroke
-			(width 0)
-			(type default)
-		)
-	)
-	(wire
-		(pts
-			(xy 200.66 90.17) (xy 200.66 96.52)
-		)
-		(stroke
-			(width 0)
-			(type default)
-		)
-	)
-	(wire
-		(pts
-			(xy 116.84 39.37) (xy 124.46 39.37)
-		)
-		(stroke
-			(width 0)
-			(type default)
-		)
-	)
-	(wire
-		(pts
-			(xy 71.12 52.07) (xy 71.12 54.61)
-		)
-		(stroke
-			(width 0)
-			(type default)
-		)
-	)
-	(wire
-		(pts
 			(xy 45.72 49.53) (xy 45.72 50.8)
 		)
@@
 	(wire
 		(pts
-			(xy 113.03 71.12) (xy 120.65 71.12)
-		)
-		(stroke
-			(width 0)
-			(type default)
-		)
-	)
-	(wire
-		(pts
 			(xy 45.72 45.72) (xy 45.72 44.45)
 		)
@@
 	(wire
 		(pts
+			(xy 76.2 109.22) (xy 113.03 109.22)
+		)
+		(stroke
+			(width 0)
+			(type default)
+		)
+	)
+	(wire
+		(pts
 			(xy 116.84 48.26) (xy 124.46 48.26)
 		)
@@
 	(wire
 		(pts
+			(xy 113.03 109.22) (xy 113.03 93.98)
+		)
+		(stroke
+			(width 0)
+			(type default)
+		)
+	)
+	(wire
+		(pts
 			(xy 50.8 45.72) (xy 45.72 45.72)
 		)
@@
 	(wire
 		(pts
+			(xy 113.03 93.98) (xy 118.11 93.98)
+		)
+		(stroke
+			(width 0)
+			(type default)
+		)
+	)
+	(wire
+		(pts
 			(xy 96.52 44.45) (xy 96.52 40.64)
 		)
@@
 		(pts
 			(xy -204.47 17.78) (xy -191.77 17.78)
-		)
-		(stroke
-			(width 0)
-			(type default)
-		)
-	)
-	(wire
-		(pts
-			(xy 113.03 71.12) (xy 113.03 76.2)
 		)
 		(stroke
@@
 	)
 	(symbol
+		(lib_id "Switch:SW_Push")
+		(at 76.2 104.14 90)
+		(unit 1)
+		(exclude_from_sim no)
+		(in_bom yes)
+		(on_board yes)
+		(dnp no)
+		(fields_autoplaced yes)
+		(property "Reference" "SW3"
+			(at 77.47 102.8699 90)
+			(effects
+				(font
+					(size 1.27 1.27)
+				)
+				(justify right)
+			)
+		)
+		(property "Value" "SW_Push"
+			(at 77.47 105.4099 90)
+			(effects
+				(font
+					(size 1.27 1.27)
+				)
+				(justify right)
+			)
+		)
+		(property "Footprint" "Button_Switch_THT:SW_Tactile_SKHH_Angled"
+			(at 71.12 104.14 0)
+			(effects
+				(font
+					(size 1.27 1.27)
+				)
+				(hide yes)
+			)
+		)
+		(property "Datasheet" "~"
+			(at 71.12 104.14 0)
+			(effects
+				(font
+					(size 1.27 1.27)
+				)
+				(hide yes)
+			)
+		)
+		(property "Description" "Push button switch, generic, two pins"
+			(at 76.2 104.14 0)
+			(effects
+				(font
+					(size 1.27 1.27)
+				)
+				(hide yes)
+			)
+		)
+		(pin "2"
+		)
+		(pin "1"
+		)
+		(instances
+			(project ""
+				(path "/cf194c5a-6388-4211-91ca-f35a7fb9ca55"
+					(reference "SW3")
+					(unit 1)
+				)
+			)
+		)
+	)
+	(symbol
 		(lib_id "power:GND")
-		(at 107.95 55.88 0)
+		(at 69.85 99.06 0)
 		(unit 1)
 		(exclude_from_sim no)
@@
 		(fields_autoplaced yes)
 		(property "Reference" "#PWR016"
-			(at 107.95 62.23 0)
+			(at 69.85 105.41 0)
 			(effects
 				(font
@@
 		)
 		(property "Value" "GND"
-			(at 107.95 60.96 0)
+			(at 69.85 104.14 0)
 			(effects
 				(font
@@
 		)
 		(property "Footprint" ""
-			(at 107.95 55.88 0)
+			(at 69.85 99.06 0)
 			(effects
 				(font
@@
 		)
 		(property "Datasheet" ""
-			(at 107.95 55.88 0)
+			(at 69.85 99.06 0)
 			(effects
 				(font
@@
 		)
 		(property "Description" "Power symbol creates a global label with name \"GND\" , ground"
-			(at 107.95 55.88 0)
+			(at 69.85 99.06 0)
 			(effects
 				(font
@@
 					(unit 1)
 				)
-			)
-		)
-	)
-	(symbol
-		(lib_name "SW_Push_Dual_1")
-		(lib_id "Switch:SW_Push_Dual")
-		(at 118.11 64.77 90)
-		(unit 1)
-		(exclude_from_sim no)
-		(in_bom yes)
-		(on_board no)
-		(dnp no)
-		(property "Reference" "SW1"
-			(at 111.76 66.0401 90)
-			(effects
-				(font
-					(size 1.27 1.27)
-				)
-				(justify left)
-			)
-		)
-		(property "Value" "SW_Push_Dual"
-			(at 111.76 63.754 90)
-			(effects
-				(font
-					(size 1.27 1.27)
-				)
-				(justify left)
-			)
-		)
-		(property "Footprint" "Button_Switch_THT:SW_SPST_Omron_B3F-50xx"
-			(at 110.49 64.77 0)
-			(effects
-				(font
-					(size 1.27 1.27)
-				)
-				(hide yes)
-			)
-		)
-		(property "Datasheet" "~"
-			(at 118.11 64.77 0)
-			(effects
-				(font
-					(size 1.27 1.27)
-				)
-				(hide yes)
-			)
-		)
-		(property "Description" "Push button switch, generic, symbol, four pins"
-			(at 118.11 64.77 0)
-			(effects
-				(font
-					(size 1.27 1.27)
-				)
-				(hide yes)
-			)
-		)
-		(pin "3"
-		)
-		(pin "4"
-		)
-		(pin "2"
-		)
-		(pin "1"
-		)
-		(instances
-			(project "schémas"
-				(path "/cf194c5a-6388-4211-91ca-f35a7fb9ca55"
-					(reference "SW1")
-					(unit 1)
-				)

Commit message: feat: changed schemas
Connections:
- net +3.3V: no longer U8.1 (IN+), U8.3 (OUT+), U9.2 (VI+)
- net GND: no longer U8.2 (IN-), U8.4 (OUT-), U9.1 (VI-)
- new net: U8.4 (OUT-), U9.1 (VI-)
- new net: U8.3 (OUT+), U9.2 (VI+)
- no-connect marks 16 -> 18
